File: cm4.kicad_sch (KiCad schematic)
At the start: 5 parts, among them U1 Compute Module 4

Commit message: PN update, BOM
Parts:
- D1: MPN (none) -> 604-APT1608SECK-AMT; PN (none) -> 604-APT1608SECK-AMT
- R1: value 1k -> 470R; MPN CRCW06031K00JNECC -> 71-CRCW0603J-470-E3; PN CRCW06031K00JNECC -> 71-CRCW0603J-470-E3
Changed lines of the file:
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@@
   (symbol (lib_id "power:+3.3V") (at 189.23 176.53 0) (unit 1)
     (in_bom yes) (on_board yes) (dnp no) (fields_autoplaced)
-    (property "Reference" "#PWR015" (at 189.23 180.34 0)
+    (property "Reference" "#PWR05" (at 189.23 180.34 0)
       (effects (font (size 1.27 1.27)) hide)
     )
@@
       (project "m17-rru-cm4"
         (path "/26152054-c498-4233-a311-ae5a54cf1383/3aa82914-11c8-4bf6-b7a9-00486758c5fe"
-          (reference "#PWR015") (unit 1)
+          (reference "#PWR05") (unit 1)
         )
       )
@@
         )
         (path "/26152054-c498-4233-a311-ae5a54cf1383/3aa82914-11c8-4bf6-b7a9-00486758c5fe"
-          (reference "C7") (unit 1)
+          (reference "C2") (unit 1)
         )
       )
@@
         )
         (path "/26152054-c498-4233-a311-ae5a54cf1383/3aa82914-11c8-4bf6-b7a9-00486758c5fe"
-          (reference "#PWR03") (unit 1)
+          (reference "#PWR04") (unit 1)
         )
       )
@@
       (effects (font (size 1.27 1.27)) hide)
     )
-    (property "PN" "" (at 80.01 100.33 90)
-      (effects (font (size 1.27 1.27)) hide)
-    )
-    (property "MPN" "" (at 80.01 100.33 90)
+    (property "PN" "604-APT1608SECK-AMT" (at 80.01 100.33 90)
+      (effects (font (size 1.27 1.27)) hide)
+    )
+    (property "MPN" "604-APT1608SECK-AMT" (at 80.01 100.33 90)
       (effects (font (size 1.27 1.27)) hide)
     )
@@
         )
         (path "/26152054-c498-4233-a311-ae5a54cf1383/3aa82914-11c8-4bf6-b7a9-00486758c5fe"
-          (reference "#PWR01") (unit 1)
+          (reference "#PWR02") (unit 1)
         )
       )
@@
       (effects (font (size 1.27 1.27)))
     )
-    (property "Value" "1k" (at 76.2 92.71 0)
+    (property "Value" "470R" (at 76.2 92.71 0)
       (effects (font (size 1.27 1.27)))
     )
@@
       (effects (font (size 1.27 1.27)) hide)
     )
-    (property "PN" "CRCW06031K00JNECC" (at 80.01 91.44 0)
-      (effects (font (size 1.27 1.27)) hide)
-    )
-    (property "MPN" "CRCW06031K00JNECC" (at 80.01 91.44 0)
+    (property "PN" "71-CRCW0603J-470-E3" (at 80.01 91.44 0)
+      (effects (font (size 1.27 1.27)) hide)
+    )
+    (property "MPN" "71-CRCW0603J-470-E3" (at 80.01 91.44 0)
       (effects (font (size 1.27 1.27)) hide)
     )
@@
         )
         (path "/26152054-c498-4233-a311-ae5a54cf1383/3aa82914-11c8-4bf6-b7a9-00486758c5fe"
-          (reference "R6") (unit 1)
+          (reference "R1") (unit 1)
         )
       )
@@
   (symbol (lib_id "power:+3.3V") (at 80.01 86.36 0) (unit 1)
     (in_bom yes) (on_board yes) (dnp no) (fields_autoplaced)
-    (property "Reference" "#PWR016" (at 80.01 90.17 0)
+    (property "Reference" "#PWR01" (at 80.01 90.17 0)
       (effects (font (size 1.27 1.27)) hide)
     )
@@
       (project "m17-rru-cm4"
         (path "/26152054-c498-4233-a311-ae5a54cf1383/3aa82914-11c8-4bf6-b7a9-00486758c5fe"
-          (reference "#PWR016") (unit 1)
+          (reference "#PWR01") (unit 1)
         )
       )
@@
         )
         (path "/26152054-c498-4233-a311-ae5a54cf1383/3aa82914-11c8-4bf6-b7a9-00486758c5fe"
-          (reference "#PWR04") (unit 1)
+          (reference "#PWR06") (unit 1)
         )
       )
@@
         )
         (path "/26152054-c498-4233-a311-ae5a54cf1383/3aa82914-11c8-4bf6-b7a9-00486758c5fe"
-          (reference "#PWR05") (unit 1)
+          (reference "#PWR07") (unit 1)
         )
       )
@@
         )
         (path "/26152054-c498-4233-a311-ae5a54cf1383/3aa82914-11c8-4bf6-b7a9-00486758c5fe"
-          (reference "#PWR02") (unit 1)
-        )
-      )
+          (reference "#PWR03") (unit 1)
+        )
+      )
