File: interfaces.kicad_sch (KiCad schematic)
At the start: 5 parts, among them J1 Conn_02x05_Odd_Even, J2 RJ45_JK0654219

Commit message: PN update, BOM
Parts:
- J1: MPN (none) -> 649-1012938391001ALF; PN (none) -> 649-1012938391001ALF
Changed lines of the file:
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@@
         )
         (path "/26152054-c498-4233-a311-ae5a54cf1383/1121b73d-0dff-4516-83a2-d497447544a0"
-          (reference "#PWR013") (unit 1)
+          (reference "#PWR010") (unit 1)
         )
       )
@@
         )
         (path "/26152054-c498-4233-a311-ae5a54cf1383/1121b73d-0dff-4516-83a2-d497447544a0"
-          (reference "#PWR06") (unit 1)
+          (reference "#PWR08") (unit 1)
         )
       )
@@
         )
         (path "/26152054-c498-4233-a311-ae5a54cf1383/1121b73d-0dff-4516-83a2-d497447544a0"
-          (reference "R4") (unit 1)
+          (reference "R2") (unit 1)
         )
       )
@@
     )
     (property "Datasheet" "~" (at 91.44 95.25 0)
+      (effects (font (size 1.27 1.27)) hide)
+    )
+    (property "MPN" "649-1012938391001ALF" (at 91.44 95.25 0)
+      (effects (font (size 1.27 1.27)) hide)
+    )
+    (property "PN" "649-1012938391001ALF" (at 91.44 95.25 0)
       (effects (font (size 1.27 1.27)) hide)
     )
@@
         )
         (path "/26152054-c498-4233-a311-ae5a54cf1383/1121b73d-0dff-4516-83a2-d497447544a0"
-          (reference "R5") (unit 1)
+          (reference "R3") (unit 1)
         )
       )
@@
         )
         (path "/26152054-c498-4233-a311-ae5a54cf1383/1121b73d-0dff-4516-83a2-d497447544a0"
-          (reference "#PWR014") (unit 1)
+          (reference "#PWR09") (unit 1)
         )
       )
@@
         )
         (path "/26152054-c498-4233-a311-ae5a54cf1383/1121b73d-0dff-4516-83a2-d497447544a0"
-          (reference "C2") (unit 1)
-        )
-      )
+          (reference "C3") (unit 1)
+        )
+      )

Commit message: WIP PCB
Parts:
- J1: footprint (none) -> Connector_PinHeader_2.54mm:PinHeader_2x05_P2.54mm_Vertical_SMD
Changed lines of the file:
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@@
       (effects (font (size 1.27 1.27)))
     )
-    (property "Footprint" "" (at 91.44 95.25 0)
+    (property "Footprint" "Connector_PinHeader_2.54mm:PinHeader_2x05_P2.54mm_Vertical_SMD" (at 91.44 95.25 0)
       (effects (font (size 1.27 1.27)) hide)
     )

Commit message: WIP PCB layout
Connections:
- net ETH_LEDG: now also R1.1; no longer R1.1
- net ETH_LEDY: now also R1.1; no longer R1.1
Other:
- company: (none) -> M17 Project
- title: (none) -> RRU CM4 board
- moved on the sheet: C2, J1, J2, R1
