File: psu.kicad_sch (KiCad schematic)
At the start: 10 parts, among them U2 TP6841

Commit message: PN update, BOM
Parts:
- renumbered C3 to C4, C4 to C5, C5 to C6, C6 to C7, R1 to R4, R2 to R5, R3 to R6
Changed lines of the file:
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@@
   (symbol (lib_id "power:GND") (at 168.91 113.03 0) (unit 1)
     (in_bom yes) (on_board yes) (dnp no) (fields_autoplaced)
-    (property "Reference" "#PWR011" (at 168.91 119.38 0)
+    (property "Reference" "#PWR015" (at 168.91 119.38 0)
       (effects (font (size 1.27 1.27)) hide)
     )
@@
       (project "m17-rru-cm4"
         (path "/26152054-c498-4233-a311-ae5a54cf1383/7c433ee8-ee3c-4f2c-88bb-a4c12c373309"
-          (reference "#PWR011") (unit 1)
+          (reference "#PWR015") (unit 1)
         )
       )
@@
   (symbol (lib_id "power:GND") (at 121.92 106.68 0) (unit 1)
     (in_bom yes) (on_board yes) (dnp no) (fields_autoplaced)
-    (property "Reference" "#PWR08" (at 121.92 113.03 0)
+    (property "Reference" "#PWR012" (at 121.92 113.03 0)
       (effects (font (size 1.27 1.27)) hide)
     )
@@
       (project "m17-rru-cm4"
         (path "/26152054-c498-4233-a311-ae5a54cf1383/7c433ee8-ee3c-4f2c-88bb-a4c12c373309"
-          (reference "#PWR08") (unit 1)
+          (reference "#PWR012") (unit 1)
         )
       )
@@
   (symbol (lib_id "Device:R_Small") (at 168.91 107.95 0) (unit 1)
     (in_bom yes) (on_board yes) (dnp no)
-    (property "Reference" "R2" (at 172.72 106.68 0)
+    (property "Reference" "R5" (at 172.72 106.68 0)
       (effects (font (size 1.27 1.27)))
     )
@@
       (project "m17-rru-cm4"
         (path "/26152054-c498-4233-a311-ae5a54cf1383/7c433ee8-ee3c-4f2c-88bb-a4c12c373309"
-          (reference "R2") (unit 1)
+          (reference "R5") (unit 1)
         )
       )
@@
   (symbol (lib_id "Device:C_Small") (at 121.92 101.6 0) (unit 1)
     (in_bom yes) (on_board yes) (dnp no) (fields_autoplaced)
-    (property "Reference" "C4" (at 124.2441 100.3942 0)
+    (property "Reference" "C5" (at 124.2441 100.3942 0)
       (effects (font (size 1.27 1.27)) (justify left))
     )
@@
       (project "m17-rru-cm4"
         (path "/26152054-c498-4233-a311-ae5a54cf1383/7c433ee8-ee3c-4f2c-88bb-a4c12c373309"
-          (reference "C4") (unit 1)
+          (reference "C5") (unit 1)
         )
       )
@@
   (symbol (lib_id "Device:C_Small") (at 162.56 83.82 90) (unit 1)
     (in_bom yes) (on_board yes) (dnp no) (fields_autoplaced)
-    (property "Reference" "C5" (at 162.5663 78.1136 90)
+    (property "Reference" "C6" (at 162.5663 78.1136 90)
       (effects (font (size 1.27 1.27)))
     )
@@
       (project "m17-rru-cm4"
         (path "/26152054-c498-4233-a311-ae5a54cf1383/7c433ee8-ee3c-4f2c-88bb-a4c12c373309"
-          (reference "C5") (unit 1)
+          (reference "C6") (unit 1)
         )
       )
@@
   (symbol (lib_id "Device:C_Polarized_Small") (at 107.95 101.6 0) (unit 1)
     (in_bom yes) (on_board yes) (dnp no) (fields_autoplaced)
-    (property "Reference" "C3" (at 110.109 99.8418 0)
+    (property "Reference" "C4" (at 110.109 99.8418 0)
       (effects (font (size 1.27 1.27)) (justify left))
     )
@@
       (project "m17-rru-cm4"
         (path "/26152054-c498-4233-a311-ae5a54cf1383/7c433ee8-ee3c-4f2c-88bb-a4c12c373309"
-          (reference "C3") (unit 1)
+          (reference "C4") (unit 1)
         )
       )
@@
   (symbol (lib_id "power:GND") (at 153.67 113.03 0) (unit 1)
     (in_bom yes) (on_board yes) (dnp no) (fields_autoplaced)
-    (property "Reference" "#PWR010" (at 153.67 119.38 0)
+    (property "Reference" "#PWR014" (at 153.67 119.38 0)
       (effects (font (size 1.27 1.27)) hide)
     )
@@
       (project "m17-rru-cm4"
         (path "/26152054-c498-4233-a311-ae5a54cf1383/7c433ee8-ee3c-4f2c-88bb-a4c12c373309"
-          (reference "#PWR010") (unit 1)
+          (reference "#PWR014") (unit 1)
         )
       )
@@
   (symbol (lib_id "Device:R_Small") (at 137.16 101.6 90) (unit 1)
     (in_bom yes) (on_board yes) (dnp no)
-    (property "Reference" "R1" (at 137.16 104.14 90)
+    (property "Reference" "R4" (at 137.16 104.14 90)
       (effects (font (size 1.27 1.27)))
     )
@@
       (project "m17-rru-cm4"
         (path "/26152054-c498-4233-a311-ae5a54cf1383/7c433ee8-ee3c-4f2c-88bb-a4c12c373309"
-          (reference "R1") (unit 1)
+          (reference "R4") (unit 1)
         )
       )
@@
   (symbol (lib_id "power:GND") (at 185.42 113.03 0) (unit 1)
     (in_bom yes) (on_board yes) (dnp no) (fields_autoplaced)
-    (property "Reference" "#PWR012" (at 185.42 119.38 0)
+    (property "Reference" "#PWR016" (at 185.42 119.38 0)
       (effects (font (size 1.27 1.27)) hide)
     )
@@
       (project "m17-rru-cm4"
         (path "/26152054-c498-4233-a311-ae5a54cf1383/7c433ee8-ee3c-4f2c-88bb-a4c12c373309"
-          (reference "#PWR012") (unit 1)
+          (reference "#PWR016") (unit 1)
         )
       )
@@
   (symbol (lib_id "power:GND") (at 107.95 106.68 0) (unit 1)
     (in_bom yes) (on_board yes) (dnp no) (fields_autoplaced)
-    (property "Reference" "#PWR07" (at 107.95 113.03 0)
+    (property "Reference" "#PWR011" (at 107.95 113.03 0)
       (effects (font (size 1.27 1.27)) hide)
     )
@@
       (project "m17-rru-cm4"
         (path "/26152054-c498-4233-a311-ae5a54cf1383/7c433ee8-ee3c-4f2c-88bb-a4c12c373309"
-          (reference "#PWR07") (unit 1)
+          (reference "#PWR011") (unit 1)
         )
       )
@@
   (symbol (lib_id "power:GND") (at 137.16 88.9 0) (unit 1)
     (in_bom yes) (on_board yes) (dnp no) (fields_autoplaced)
-    (property "Reference" "#PWR09" (at 137.16 95.25 0)
+    (property "Reference" "#PWR013" (at 137.16 95.25 0)
       (effects (font (size 1.27 1.27)) hide)
     )
@@
       (project "m17-rru-cm4"
         (path "/26152054-c498-4233-a311-ae5a54cf1383/7c433ee8-ee3c-4f2c-88bb-a4c12c373309"
-          (reference "#PWR09") (unit 1)
+          (reference "#PWR013") (unit 1)
         )
       )
@@
   (symbol (lib_id "Device:C_Small") (at 185.42 107.95 180) (unit 1)
     (in_bom yes) (on_board yes) (dnp no) (fields_autoplaced)
-    (property "Reference" "C6" (at 187.7441 106.7315 0)
+    (property "Reference" "C7" (at 187.7441 106.7315 0)
       (effects (font (size 1.27 1.27)) (justify right))
     )
@@
       (project "m17-rru-cm4"
         (path "/26152054-c498-4233-a311-ae5a54cf1383/7c433ee8-ee3c-4f2c-88bb-a4c12c373309"
-          (reference "C6") (unit 1)
+          (reference "C7") (unit 1)
         )
       )
@@
   (symbol (lib_id "Device:R_Small") (at 177.8 101.6 90) (unit 1)
     (in_bom yes) (on_board yes) (dnp no)
-    (property "Reference" "R3" (at 177.8 104.14 90)
+    (property "Reference" "R6" (at 177.8 104.14 90)
       (effects (font (size 1.27 1.27)))
     )
@@
       (project "m17-rru-cm4"
         (path "/26152054-c498-4233-a311-ae5a54cf1383/7c433ee8-ee3c-4f2c-88bb-a4c12c373309"
-          (reference "R3") (unit 1)
-        )
-      )
+          (reference "R6") (unit 1)
+        )
+      )

Commit message: WIP PCB layout
Parts:
- TP1: now left out of the parts list
Other:
- company: (none) -> M17 Project
- title: (none) -> RRU CM4 board
- moved on the sheet: C4, C5, C6, C7, L1, R4, R5, R6, TP1, U2
