File: m17-rru-cm4.kicad_pcb (KiCad board)
At the start: 2 copper layers, 95 x 62 mm, 24 parts, among them J1 Conn_02x05_Odd_Even, J2 RJ45_JK0654219, U1 Compute Module 4, U2 TP6841

Commit message: missing comma
Other:
- board text added: "RRU Interface Board Wojciech Kaczmarski, SP5WWP M17 Project, January 2024"
- board text removed: "RRU Interface Board Wojciech Kaczmarski SP5WWP M17 Project, January 2024"
Changed lines of the file:
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@@
     (effects (font (size 1 1) (thickness 0.15)) (justify right bottom))
   )
-  (gr_text "RRU Interface Board\nWojciech Kaczmarski SP5WWP\nM17 Project, January 2024" (at 107.442 96.266 90) (layer "F.SilkS")
+  (gr_text "RRU Interface Board\nWojciech Kaczmarski, SP5WWP\nM17 Project, January 2024" (at 107.442 96.266 90) (layer "F.SilkS")
     (effects (font (size 1 1) (thickness 0.15)) (justify left bottom))
   )
